File: schematic/user/ezDV.kicad_sch (KiCad schematic)
At the start: 0 parts

Commit message: v0.4 board submitted for build/assembly.
Other:
- company: (none) -> FreeDV Project
- title: (none) -> ezDV
Changed lines of the file:
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@@
 (kicad_sch (version 20211123) (generator eeschema)
   (paper "A4")
+  (title_block
+    (title "ezDV")
+    (date "2022-10-01")
+    (rev "v0.4")
+    (company "FreeDV Project")
+  )
   (sheet (at 77.47 30.48) (size 41.91 27.94) (fields_autoplaced)
     (stroke (width 0.1524) (type solid) (color 0 0 0 0))
